File: src/solder.kicad_pcb (KiCad board)
At the start: 2 copper layers, 40 x 96 mm, 39 parts, among them Q1 BC337, Q2 BC337, Q3 BC337, Q4 BC337, Q5 BC337, Q6 BC337, Q7 BC337, Q8 BC337, SW1 SW_Push, SW2 SW_Push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

Commit message: Add files via upload
Parts:
- added G***: LOGO, LOGO, B.Cu at (50.6, 105.4)
Other:
- outline, holes or cut-outs redrawn
